Commit message: Modify description

File: eric_a_description/urdf/eric_a.urdf.xacro (robot description, xacro)
@@ -86,5 +86,5 @@
       </geometry>
     </collision>
-  </link> <!--wheel_left_joint-->
+  </link> <!--wheel_left_link-->
   <joint
     name="wheel_left_joint"
@@ -139,5 +139,5 @@
       </geometry>
     </collision>
-  </link> <!--wheel_right_joint-->
+  </link> <!--wheel_right_link-->
   <joint
     name="wheel_right_joint"
@@ -152,5 +152,5 @@
     <axis
       xyz="0 1 0" />
-  </joint>
+  </joint> <!--wheel right joint-->
   <link
     name="base_scan">
@@ -206,3 +206,17 @@
       xyz="0 0 0" />
   </joint>
+  <link name="imu_link">
+      <visual>
+        <origin xyz="0 0 0" rpy="0 0 0" />
+        <geometry>
+          <box size="0.01 0.01 0.01" />
+        </geometry>
+        <material name="" />
+      </visual>
+  </link>
+  <joint name="base_link_to_imu_link" type="fixed">
+    <origin xyz="0.0 0 0.2" rpy="0 0 0" />
+    <parent link="base_link"/>
+    <child link="imu_link" />
+  </joint>
 </robot>
